Commit message: Added gazebo models and worlds

File: neos_description/urdf/neos.urdf (robot description, URDF)
Before this commit: robot neos, 5 links, 4 joints
Joints:
- joint left_wheel_joint: origin xyz=0 0.15 -0.05 rpy=1.5708 0 0 -> xyz=0 0.15 -0.025 rpy=1.5708 0 0
- joint right_wheel_joint: origin xyz=0 -0.15 -0.05 rpy=1.5708 0 0 -> xyz=0 -0.15 -0.025 rpy=1.5708 0 0

File: neos_description/urdf/neos.xacro (robot description, xacro)
@@ -55,5 +55,5 @@
       <parent link="base_link"/>
       <child link="${name}"/>
-      <origin xyz="0 ${side * wheel_separation/2} -${wheel_radius}" rpy="1.5708 0 0"/>
+      <origin xyz="0 ${side * wheel_separation/2} -${wheel_radius/2}" rpy="1.5708 0 0"/>
       <axis xyz="0 0 1"/>
     </joint>
@@ -83,5 +83,5 @@
       <parent link="base_link"/>
       <child link="${name}"/>
-      <origin xyz="${x_pos} 0 -${caster_radius}" rpy="0 0 0"/>
+      <origin xyz="${x_pos} 0 -0.03" rpy="0 0 0"/>
     </joint>
   </xacro:macro>

Commit message: added docs

File: neos_description/urdf/neos.urdf (robot description, URDF)
Before this commit: robot neos, 5 links, 4 joints
Joints:
- joint front_caster_joint: origin xyz=0.15 0 -0.03 rpy=0 0 0 -> xyz=0.15 0 -0.025 rpy=0 0 0
- joint rear_caster_joint: origin xyz=-0.15 0 -0.03 rpy=0 0 0 -> xyz=-0.15 0 -0.025 rpy=0 0 0

File: neos_description/urdf/neos.xacro (robot description, xacro)
@@ -83,5 +83,5 @@
       <parent link="base_link"/>
       <child link="${name}"/>
-      <origin xyz="${x_pos} 0 -0.03" rpy="0 0 0"/>
+      <origin xyz="${x_pos} 0 -0.04" rpy="0 0 0"/>
     </joint>
   </xacro:macro>

Commit message: aligning wheels with caster wheels

File: neos_description/urdf/neos.urdf (robot description, URDF)
Before this commit: robot neos, 5 links, 4 joints
Joints:
- joint front_caster_joint: origin xyz=0.15 0 -0.025 rpy=0 0 0 -> xyz=0.15 0 -0.04 rpy=0 0 0
- joint rear_caster_joint: origin xyz=-0.15 0 -0.025 rpy=0 0 0 -> xyz=-0.15 0 -0.04 rpy=0 0 0

Commit message: fixed wheels / caster wheel alignement

File: neos_description/urdf/neos.urdf (robot description, URDF)
Before this commit: robot neos, 5 links, 4 joints
Joints:
- joint front_caster_joint: origin xyz=0.15 0 -0.04 rpy=0 0 0 -> xyz=0.15 0 -0.044 rpy=0 0 0
- joint left_wheel_joint: origin xyz=0 0.15 -0.025 rpy=1.5708 0 0 -> xyz=0 -0.15 -0.025 rpy=1.5708 0 0
- joint rear_caster_joint: origin xyz=-0.15 0 -0.04 rpy=0 0 0 -> xyz=-0.15 0 -0.044 rpy=0 0 0
- joint right_wheel_joint: origin xyz=0 -0.15 -0.025 rpy=1.5708 0 0 -> xyz=0 0.15 -0.025 rpy=1.5708 0 0

File: neos_description/urdf/neos.xacro (robot description, xacro)
@@ -83,10 +83,10 @@
       <parent link="base_link"/>
       <child link="${name}"/>
-      <origin xyz="${x_pos} 0 -0.04" rpy="0 0 0"/>
+      <origin xyz="${x_pos} 0 -0.044" rpy="0 0 0"/>
     </joint>
   </xacro:macro>
   <!-- Create Wheels -->
-  <xacro:wheel name="left_wheel" side="1"/>
-  <xacro:wheel name="right_wheel" side="-1"/>
+  <xacro:wheel name="left_wheel" side="-1"/>
+  <xacro:wheel name="right_wheel" side="1"/>
   <!-- Create Casters -->
   <xacro:caster name="front_caster" x_pos="0.15"/>

Commit message: Adjust acceleration and velocity values

File: neos_description/urdf/neos.urdf (robot description, URDF)
Before this commit: robot neos, 5 links, 4 joints
Links:
- link base_link: mass 10 -> 5

File: neos_description/urdf/neos.xacro (robot description, xacro)
@@ -8,5 +8,5 @@
   <xacro:property name="wheel_separation" value="0.3"/>
   <xacro:property name="caster_radius" value="0.03"/>
-  <xacro:property name="base_mass" value="10"/>
+  <xacro:property name="base_mass" value="5"/>
   <xacro:property name="wheel_mass" value="0.5"/>
   <xacro:property name="caster_mass" value="0.1"/>

Commit message: Added Lidar

File: neos_description/urdf/neos.urdf (robot description, URDF)
Before this commit: robot neos, 5 links, 4 joints
Links:
- added link lidar_link, mass 0.1; collision cylinder length=0.05 radius=0.05; visual cylinder length=0.05 radius=0.05
Joints:
- added joint lidar_joint: type fixed, parent base_link, child lidar_link, origin xyz=0 0 0.09 rpy=0 0 0
- joint front_caster_joint: origin xyz=0.15 0 -0.044 rpy=0 0 0 -> xyz=0.15 0 -0.048 rpy=0 0 0
- joint rear_caster_joint: origin xyz=-0.15 0 -0.044 rpy=0 0 0 -> xyz=-0.15 0 -0.048 rpy=0 0 0

File: neos_description/urdf/neos.xacro (robot description, xacro)
@@ -95,6 +95,6 @@
   <xacro:caster name="rear_caster" x_pos="-0.15"/>
   <!-- Add LiDAR Sensor (using default parameters) -->
-  <xacro:neos_lidar/>
+  <!-- <xacro:neos_lidar/> -->
   <!-- Alternative: Add LiDAR with custom parameters -->
-  <!-- <xacro:neos_lidar parent_link="base_link" x="0" y="0" z="0.25" topic="/scan" update_rate="30" min_range="0.1" max_range="5.0" samples="360"/> -->
+  <xacro:neos_lidar parent_link="base_link" x="0" y="0" z="0.09"/>
 </robot>

File: neos_description/urdf/neos_lidar.xacro (robot description, xacro)
@@ -30,11 +30,11 @@
       <origin xyz="${x} ${y} ${z}" rpy="0 0 0"/>
     </joint>
-    <!-- Gazebo LiDAR Plugin -->
+    <!-- Gazebo Sim LiDAR Sensor -->
     <gazebo reference="lidar_link">
-      <sensor type="ray" name="lidar_sensor">
+      <sensor name="lidar_sensor" type="lidar">
         <pose>0 0 0 0 0 0</pose>
         <visualize>true</visualize>
         <update_rate>${update_rate}</update_rate>
-        <ray>
+        <lidar>
           <scan>
             <horizontal>
@@ -55,10 +55,7 @@
             <stddev>0.01</stddev>
           </noise>
-        </ray>
-        <plugin filename="libgazebo_ros_ray_sensor.so" name="lidar_plugin">
-          <ros>
-            <remapping>~/out:=${topic}</remapping>
-          </ros>
-          <output_type>sensor_msgs/LaserScan</output_type>
+        </lidar>
+        <plugin filename="gz-sim-lidar-system" name="gz::sim::systems::Lidar">
+          <topic>${topic}</topic>
           <frame_name>lidar_link</frame_name>
         </plugin>

Commit message: Fixed robot driving direction and lidar config

File: neos_description/urdf/neos.urdf (robot description, URDF)
Before this commit: robot neos, 6 links, 5 joints
Joints:
- joint front_caster_joint: origin xyz=0.15 0 -0.048 rpy=0 0 0 -> xyz=0.15 0 -0.04499 rpy=0 0 0
- joint left_wheel_joint: axis 0 0 1 -> 0 0 -1; origin xyz=0 -0.15 -0.025 rpy=1.5708 0 0 -> xyz=0 0.15 -0.025 rpy=1.5708 0 0
- joint rear_caster_joint: origin xyz=-0.15 0 -0.048 rpy=0 0 0 -> xyz=-0.15 0 -0.04499 rpy=0 0 0
- joint right_wheel_joint: axis 0 0 1 -> 0 0 -1; origin xyz=0 0.15 -0.025 rpy=1.5708 0 0 -> xyz=0 -0.15 -0.025 rpy=1.5708 0 0

File: neos_description/urdf/neos.xacro (robot description, xacro)
@@ -58,5 +58,5 @@
       <child link="${name}"/>
       <origin xyz="0 ${side * wheel_separation/2} -${wheel_radius/2}" rpy="1.5708 0 0"/>
-      <axis xyz="0 0 1"/>
+      <axis xyz="0 0 -1"/>
     </joint>
   </xacro:macro>
@@ -85,10 +85,10 @@
       <parent link="base_link"/>
       <child link="${name}"/>
-      <origin xyz="${x_pos} 0 -0.048" rpy="0 0 0"/>
+      <origin xyz="${x_pos} 0 -0.04499" rpy="0 0 0"/>
     </joint>
   </xacro:macro>
   <!-- Create Wheels -->
-  <xacro:wheel name="left_wheel" side="-1"/>
-  <xacro:wheel name="right_wheel" side="1"/>
+  <xacro:wheel name="left_wheel" side="1"/>
+  <xacro:wheel name="right_wheel" side="-1"/>
   <!-- Create Casters -->
   <xacro:caster name="front_caster" x_pos="0.15"/>

File: neos_description/urdf/neos_lidar.xacro (robot description, xacro)
@@ -2,5 +2,5 @@
 <robot xmlns:xacro="http://www.ros.org/wiki/xacro" name="neos_lidar">
   <!-- Parameterized LiDAR Sensor Macro -->
-  <xacro:macro name="neos_lidar" params="parent_link:=base_link x:=0 y:=0 z:=0.2 topic:=/scan update_rate:=30 min_range:=0.12 max_range:=3.5 samples:=720">
+  <xacro:macro name="neos_lidar" params="parent_link:=base_link x:=0 y:=0 z:=0.2 topic:=/scan update_rate:=30 min_range:=0.1 max_range:=7.0 samples:=720">
     <!-- LiDAR Link -->
     <link name="lidar_link">
@@ -32,9 +32,10 @@
     <!-- Gazebo Sim LiDAR Sensor -->
     <gazebo reference="lidar_link">
-      <sensor name="lidar_sensor" type="lidar">
+      <sensor name="lidar_sensor" type="gpu_lidar">
         <pose>0 0 0 0 0 0</pose>
+        <topic>${topic}</topic>
+        <update_rate>${update_rate}</update_rate>
         <visualize>true</visualize>
-        <update_rate>${update_rate}</update_rate>
-        <lidar>
+        <ray>
           <scan>
             <horizontal>
@@ -44,4 +45,10 @@
               <max_angle>1.5708</max_angle>
             </horizontal>
+            <vertical>
+              <samples>1</samples>
+              <resolution>0.01</resolution>
+              <min_angle>0</min_angle>
+              <max_angle>0</max_angle>
+            </vertical>
           </scan>
           <range>
@@ -55,9 +62,6 @@
             <stddev>0.01</stddev>
           </noise>
-        </lidar>
-        <plugin filename="gz-sim-lidar-system" name="gz::sim::systems::Lidar">
-          <topic>${topic}</topic>
-          <frame_name>lidar_link</frame_name>
-        </plugin>
+        </ray>
+        <always_on>1</always_on>
       </sensor>
     </gazebo>
